File: electrical/norbert/v1/norbert_v1/norbert_v1.kicad_sch (KiCad schematic)
At the start: 23 parts, among them J1 PPTC191LFBN-RC, J2 PPTC191LFBN-RC, J3 61300411121, J4 61300411121, U1 ESP32-DevKitC, U2 SN74LVC1T45DCKR, U3 SN74LVC1T45DCKR

Commit message: Add remaining changes for electrical design
Parts:
- TB1, TB2, TB3, TB4, TB5, TB6, TB7: footprint (none) -> LIB_5442248:5442248
Changed lines of the file:
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@@
       (effects (font (size 1.27 1.27)) (justify left))
     )
-    (property "Footprint" "" (at 187.96 31.75 0)
+    (property "Footprint" "LIB_5442248:5442248" (at 187.96 31.75 0)
       (effects (font (size 1.27 1.27)) hide)
     )
@@
       (effects (font (size 1.27 1.27)) (justify left))
     )
-    (property "Footprint" "" (at 187.96 60.96 0)
+    (property "Footprint" "LIB_5442248:5442248" (at 187.96 60.96 0)
       (effects (font (size 1.27 1.27)) hide)
     )
@@
       (effects (font (size 1.27 1.27)) (justify left))
     )
-    (property "Footprint" "" (at 187.96 81.28 0)
+    (property "Footprint" "LIB_5442248:5442248" (at 187.96 81.28 0)
       (effects (font (size 1.27 1.27)) hide)
     )
@@
       (effects (font (size 1.27 1.27)) (justify left))
     )
-    (property "Footprint" "" (at 187.96 20.32 0)
+    (property "Footprint" "LIB_5442248:5442248" (at 187.96 20.32 0)
       (effects (font (size 1.27 1.27)) hide)
     )
@@
       (effects (font (size 1.27 1.27)) (justify left))
     )
-    (property "Footprint" "" (at 187.96 72.39 0)
+    (property "Footprint" "LIB_5442248:5442248" (at 187.96 72.39 0)
       (effects (font (size 1.27 1.27)) hide)
     )
@@
       (effects (font (size 1.27 1.27)) (justify left))
     )
-    (property "Footprint" "" (at 187.96 52.07 0)
+    (property "Footprint" "LIB_5442248:5442248" (at 187.96 52.07 0)
       (effects (font (size 1.27 1.27)) hide)
     )
@@
       (effects (font (size 1.27 1.27)) (justify left))
     )
-    (property "Footprint" "" (at 187.96 40.64 0)
-      (effects (font (size 1.27 1.27)) hide)
-    )
+    (property "Footprint" "LIB_5442248:5442248" (at 187.96 40.64 0)
+      (effects (font (size 1.27 1.27)) hide)
+    )
