File: electrical/norbert/v1/norbert_v1/norbert_v1_pg2.kicad_sch (KiCad schematic)
At the start: 55 parts, among them J1 61300311121, J10 61300311121, J13 61300411121, J2 61300311121, J3 61300311121, J4 61300311121, J5 61300311121, J6 61300311121, J7 61300311121, J8 61300311121, J9 61300311121, U2 A4988SETTR-T, U7 PCA9685PW_112, U8 LTC2497CUHF-PBF

Commit message: Add remaining changes for electrical design
Parts:
- TB1: footprint (none) -> LIB_5442248:5442248
Changed lines of the file:
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@@
       (effects (font (size 1.27 1.27)) (justify left))
     )
-    (property "Footprint" "" (at 255.27 128.27 0)
+    (property "Footprint" "LIB_5442248:5442248" (at 255.27 128.27 0)
       (effects (font (size 1.27 1.27)) hide)
     )
@@
       (effects (font (size 1.27 1.27)) (justify left))
     )
-    (property "Footprint" "" (at 255.27 118.11 0)
-      (effects (font (size 1.27 1.27)) hide)
-    )
+    (property "Footprint" "LIB_5442248:5442248" (at 255.27 118.11 0)
+      (effects (font (size 1.27 1.27)) hide)
+    )
