File: electrical/norbert/v1/norbert_v1/norbert_v1_pg3.kicad_sch (KiCad schematic)
At the start: 33 parts, among them U3 LP2985-33DBVR, U4 LP2985-50DBVR, U9 ADP1711AUJZ-0.75R7, X1 YIZHET_LM2596_VREG, X2 YIZHET_LM2596_VREG, X3 YIZHET_LM2596_VREG, X4 YIZHET_LM2596_VREG, X5 YIZHET_LM2596_VREG

Commit message: Add remaining changes for electrical design
Parts:
- TB4: footprint (none) -> LIB_1730502:1730502
Changed lines of the file:
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@@
       (effects (font (size 1.27 1.27)) (justify left))
     )
-    (property "Footprint" "" (at 110.49 118.11 0)
+    (property "Footprint" "LIB_1730502:1730502" (at 110.49 118.11 0)
       (effects (font (size 1.27 1.27)) hide)
     )
